File: project/DemoBoard.brd (EAGLE design)
At the start: 100 x 80 mm, 50 parts, among them J1 SAMTEC-MMS-105-02-X-SVJ, J4 10104111-0001LF, U1 SN74LVC2T45YZPR, U2 STM32F207ZGT6, U3 SN74LVC2T45YZPR, U4 SN74LVC2T45YZPR, Y1 SIT1602BI-23-18E-33.333300G, Y2 SIT1602BI-23-18E-33.333300G, Y3 SIT1602BI-23-18E-33.333300G

Commit message: Add files via upload
Parts:
- moved R_OSC1 98.3 mm to (2.54, 52.1)
- moved R_OSC10 98.3 mm to (12.7, 52.1)
- moved R_OSC9 98.3 mm to (16.5, 61.0)
- moved R_PG 98.3 mm to (-15.2, 61.0)
- moved R_PG1 98.3 mm to (7.62, 61.0)
- moved C_C1 98.3 mm to (17.8, 73.7)
- moved C_C2 98.3 mm to (11.4, 73.7)
- moved C_F 98.3 mm to (53.3, 73.7)
- moved C_F1 98.3 mm to (45.7, 73.7)
- moved C_IN 98.3 mm to (38.1, 73.7)
- moved C_IN1 98.3 mm to (30.5, 73.7)
- moved C_OUT 98.3 mm to (-17.8, 67.3)
- moved C_OUT1 98.3 mm to (26.7, 67.3)
- moved C_SS 98.3 mm to (24.1, 73.7)
- moved C_SS1 98.3 mm to (61.0, 73.7)
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Other:
- board size 100 x 80 mm -> 166 x 80 mm
